File: Nixie_Clock/nixie_clk_ucontroller.sch (KiCad schematic (older format))
At the start: 0 parts

Commit message: Almost done with uC page
Parts:
- added C? (x2): C, symbol C
- added C?: 1uF, symbol C
- added C? (x3): 100nF, symbol C
- added C?: 10uF, symbol C
- added D?: LED 1, symbol LED
- added D?: LED 2, symbol LED
- added J?: Conn_01x04, symbol Conn_01x04
- added R? (x3): 10K, symbol R
- added U?: SAMD20E14A-AU, TQFP32, symbol SAMD20E14A-AU
- added Y?: Crystal, symbol Crystal
Connections:
- new net: C?.1, U?.1 (XIN32/TC2WO0/SERCOM1P0/PA00), Y?.2
- new net: C?.1, U?.2 (XOUT32/TC2WO1/SERCOM1P1/PA01), Y?.1
- new net: C?.1, U?.29 (VDDCORE)
- new net: D?.1 (K), R?.1 (x2)
- new net GND: C?.2, C?.2, C?.2, C?.2, C?.2, C?.2, C?.2, U?.10 (GND), U?.28 (GND)
- new net PA08: U?.11 (TC0WO0/SERCOM2P0/SERCOM0P0/X0/AIN16/NMI/PA08)
- new net PA09: U?.12 (TC0WO1/SERCOM2P1/SERCOM0P1/X1/AIN17/PA09)
- new net PA10: U?.13 (GCLKIO4/TC1WO0/SERCOM2P2/SERCOM0P2/X2/AIN18/PA10)
- new net PA11: U?.14 (GCLKIO5/TC1WO1/SERCOM2P3/SERCOM0P3/X3/AIN19/PA11)
- new net PA18: R?.2, U?.19 (ACCMP0/TC3WO0/SERCOM3P2/SERCOM1P2/X6/PA18)
- new net PA19: R?.2, U?.20 (ACCMP1/TC3WO1/SERCOM3P3/SERCOM1P3/X7/PA19)
- new net PA25: U?.24 (TC5WO1/SERCOM5P3/SERCOM3P3/PA25)
- new net PA27: U?.25 (GCLKIO0/PA27)
- new net PA28: U?.27 (GCLKIO0/PA28)
- new net PP3V3: C?.1, C?.1, C?.1, D?.2 (A), D?.2 (A), R?.1, U?.30 (VDDIN), U?.9 (VDDANA)
- new net TC0WO0: U?.5 (TC0WO0/SERCOM0P0/Y2/AIN0/AIN4/VREFB/PA04)
- new net TC0WO1: U?.6 (TC0W01/SERCOM0P1/Y3/AIN1/AIN5/PA05)
- new net TC1WO0: U?.7 (TC1WO0/SERCOM0P2/Y4/AIN2/AIN6/PA06)
- new net TC1WO1: U?.8 (TC1WO1/SERCOM0P3/Y5/AIN3/AIN7/PA07)
- new net TC2WO0: U?.17 (GCLKIO2/TC2WO0/SERCOM3P0/SERCOM1P0/X4/PA16)
- new net TC2WO1: U?.18 (GCLKIO3/TC2WO1/SERCOM3P1/SERCOM1P1/X5/PA17)
- new net TC3WO0: U?.15 (XIN/GCLKIO0/TC3WO0/SERCOM4P2/SERCOM2P2/PA14)
- new net TC3WO1: U?.16 (XOUT/GCLKIO1/TC3WO1/SERCOM4P3/SERCOM2P3/PA15)
- new net TC4WO0: U?.21 (GCLKIO6/TC4WO0/SERCOM5P0/SERCOM3P0/X10/PA22)
- new net TC4WO1: U?.22 (GCLKIO7/TC4WO1/SERCOM5P1/SERCOM3P1/X11/PA23)
- new net TC5WO0: U?.23 (TC5WO0/SERCOM5P2/SERCOM3P2/PA24)
- new net Y0_H: U?.3 (VOUT/Y0/AIN0/PA02)
- new net Y1_M: U?.4 (Y1/AIN1/VREFA/VREFP/PA03)
- new net ~RESET: C?.1, R?.2, U?.26 (~RESET~)
