File: Nixie_Clock/nixie_clk_5V_power.sch (KiCad schematic (older format))
At the start: 15 parts

Commit message: Sync remote
Parts:
- added C? (x2): 100nF, symbol C
- added D?: TL431D, Housings_SOIC:SOIC-8_3.9x4.9mm_Pitch1.27mm, symbol TL431D
- added R?: 10k', Resistors_SMD:R_1206, symbol R
- added R?: 10k, Resistors_SMD:R_1206, symbol R
- added R? (x2): 4.7k, Resistors_SMD:R_1206, symbol R
- C?: value CP1 -> 150u
- R?: value 68.1k -> 4.7k; Voltage 200V -> (none)
Connections:
- net GND: now also U?.2, D?.2 (A), D?.3 (A), D?.6 (A), D?.7 (A), R?.2
- net PP5V: no longer C?.1, C?.1, C?.1, R?.1, T?.4 (S2)
- net at R?.2, U?.1: now also C?.1, D?.1 (K), R?.2, R?.2
- new net: R?.1, R?.1
- new net: C?.2, C?.2, D?.8 (REF), R?.1, R?.2
- new net: C?.1, R?.1
